File: Hardware/NekoPurrTech_TiltingCtrl.kicad_sch (KiCad schematic)
At the start: 33 parts, among them IC1 TPS70933DRVR, IC2 TB67H450FNG, IC3 TPS70933DRVR, J1 Power_IN, J2 FMU_PWM, J3 Motor, J4 Dbg_Port, U1 STM32F030F4Px

Commit message: Finished Hardware
Parts:
- J4: footprint (none) -> SamacSys_Parts:Dbg_Port
Changed lines of the file:
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@@
 		)
 		(instances
-			(project ""
+			(project "NekoPurrTech_TiltingCtrl"
 				(path "/d0aecbef-76a5-4374-b49f-e202fe34b8e5"
 					(reference "R9")
@@
 		)
 		(instances
-			(project ""
+			(project "NekoPurrTech_TiltingCtrl"
 				(path "/d0aecbef-76a5-4374-b49f-e202fe34b8e5"
 					(reference "#PWR021")
@@
 		)
 		(instances
-			(project ""
+			(project "NekoPurrTech_TiltingCtrl"
 				(path "/d0aecbef-76a5-4374-b49f-e202fe34b8e5"
 					(reference "IC1")
@@
 		)
 		(instances
-			(project ""
+			(project "NekoPurrTech_TiltingCtrl"
 				(path "/d0aecbef-76a5-4374-b49f-e202fe34b8e5"
 					(reference "C4")
@@
 		)
 		(instances
-			(project ""
+			(project "NekoPurrTech_TiltingCtrl"
 				(path "/d0aecbef-76a5-4374-b49f-e202fe34b8e5"
 					(reference "#PWR04")
@@
 		)
 		(instances
-			(project ""
+			(project "NekoPurrTech_TiltingCtrl"
 				(path "/d0aecbef-76a5-4374-b49f-e202fe34b8e5"
 					(reference "U1")
@@
 		)
 		(instances
-			(project ""
+			(project "NekoPurrTech_TiltingCtrl"
 				(path "/d0aecbef-76a5-4374-b49f-e202fe34b8e5"
 					(reference "#PWR03")
@@
 		)
 		(instances
-			(project ""
+			(project "NekoPurrTech_TiltingCtrl"
 				(path "/d0aecbef-76a5-4374-b49f-e202fe34b8e5"
 					(reference "D1")
@@
 		)
 		(instances
-			(project ""
+			(project "NekoPurrTech_TiltingCtrl"
 				(path "/d0aecbef-76a5-4374-b49f-e202fe34b8e5"
 					(reference "J2")
@@
 		)
 		(instances
-			(project ""
+			(project "NekoPurrTech_TiltingCtrl"
 				(path "/d0aecbef-76a5-4374-b49f-e202fe34b8e5"
 					(reference "R6")
@@
 		)
 		(instances
-			(project ""
+			(project "NekoPurrTech_TiltingCtrl"
 				(path "/d0aecbef-76a5-4374-b49f-e202fe34b8e5"
 					(reference "#PWR018")
@@
 			)
 		)
-		(property "Footprint" ""
+		(property "Footprint" "SamacSys_Parts:Dbg_Port"
 			(at 132.08 180.34 0)
 			(effects
@@
 		)
 		(instances
-			(project ""
+			(project "NekoPurrTech_TiltingCtrl"
 				(path "/d0aecbef-76a5-4374-b49f-e202fe34b8e5"
 					(reference "C12")
@@
 		)
 		(instances
-			(project ""
+			(project "NekoPurrTech_TiltingCtrl"
 				(path "/d0aecbef-76a5-4374-b49f-e202fe34b8e5"
 					(reference "J3")
@@
 		)
 		(instances
-			(project ""
+			(project "NekoPurrTech_TiltingCtrl"
 				(path "/d0aecbef-76a5-4374-b49f-e202fe34b8e5"
 					(reference "IC2")
@@
 		)
 		(instances
-			(project ""
+			(project "NekoPurrTech_TiltingCtrl"
 				(path "/d0aecbef-76a5-4374-b49f-e202fe34b8e5"
 					(reference "R1")
@@
 		)
 		(instances
-			(project ""
+			(project "NekoPurrTech_TiltingCtrl"
 				(path "/d0aecbef-76a5-4374-b49f-e202fe34b8e5"
 					(reference "C2")
@@
 		)
 		(instances
-			(project ""
+			(project "NekoPurrTech_TiltingCtrl"
 				(path "/d0aecbef-76a5-4374-b49f-e202fe34b8e5"
 					(reference "J1")
